File: ap2112m-txb0104-module.kicad_pcb (KiCad board)
At the start: 2 copper layers, 0 parts

Commit message: Component placement, outline, no routing
Parts:
- added C1: 1u, local_footprints:1206_HS, F.Cu at (149.4, 86.4)
- added C2: 1u, local_footprints:1206_HS, F.Cu at (149.4, 91.4)
- added C3: 0.1u, local_footprints:0805_HS, F.Cu at (158.0, 86.6)
- added C4: 0.1u, local_footprints:0805_HS, F.Cu at (158.0, 91.2)
- added D1: D_Schottky, local_footprints:1206_Diode_HS, F.Cu at (146.1, 82.5)
- added J1: USB_B_Micro, local_footprints:USB-micro-B_4-legs_Banggood, F.Cu at (139.7, 88.3)
- added J10: SIG_HV, local_footprints:Pin_Header_Straight_1x04_Pitch2.54mm, F.Cu at (161.3, 82.5)
- added J11: SIG_LV, local_footprints:Pin_Header_Straight_1x04_Pitch2.54mm, F.Cu at (161.3, 95.2)
- added J2: VIN_HV, local_footprints:Pin_Header_Straight_1x01_Pitch2.54mm, F.Cu at (153.7, 82.5)
- added J3: VIN_HV, local_footprints:Pin_Header_Straight_1x01_Pitch2.54mm, F.Cu at (151.1, 82.5)
- added J4: GND, local_footprints:Pin_Header_Straight_1x01_Pitch2.54mm, F.Cu at (158.8, 82.5)
- added J5: GND, local_footprints:Pin_Header_Straight_1x01_Pitch2.54mm, F.Cu at (156.2, 82.5)
- added J6: VOUT_LV, local_footprints:Pin_Header_Straight_1x01_Pitch2.54mm, F.Cu at (153.7, 95.2)
- added J7: VOUT_LV, local_footprints:Pin_Header_Straight_1x01_Pitch2.54mm, F.Cu at (151.1, 95.2)
- added J8: GND, local_footprints:Pin_Header_Straight_1x01_Pitch2.54mm, F.Cu at (158.8, 95.2)
- added J9: GND, local_footprints:Pin_Header_Straight_1x01_Pitch2.54mm, F.Cu at (156.2, 95.2)
- added JP1: 0 Ohm, local_footprints:0805_HS, F.Cu at (146.9, 86.4)
- added JST_PH_BAT1: JST_PH_BAT, local_footprints:JST_PH_S2B-PH-K_02x2.00mm_Angled_WiderHole, F.Cu at (170.2, 89.9)
- added R1: 10k, local_footprints:0805_HS, B.Cu at (166.1, 88.4)
- added SW1: SW_REG, local_footprints:Conn_01x03_small, F.Cu at (144.1, 95.2)
- added U1: AP2112M-8SOIC, local_footprints:SOIC-8_3.9x4.9mm_Pitch1.27mm_HS, F.Cu at (153.4, 88.9)
- added U2: TXB0104, local_footprints:SOIC-14_3.9x8.7mm_Pitch1.27mm_HS, F.Cu at (163.8, 88.9)
Other:
- board outline added: 31.8 x 15.2 mm
- net class Default: via_dia 0.6096 -> 0.6858; via_drill 0.3048 -> 0.3302
- rule pad_to_mask_clearance: 0.051 -> 0.0508
- rule solder_mask_min_width: 0.25 -> 0.1016
- rule via_min_drill: 0.3048 -> 0.3302
- rule via_min_size: 0.6096 -> 0.6858
- board text added: "OFF"
- board text added: "ON"
