File: ap2112m-txb0104-module.kicad_pcb (KiCad board)
At the start: 2 copper layers, 31.8 x 15.2 mm, 22 parts, among them J1 USB_B_Micro, J10 SIG_HV, J11 SIG_LV, J2 VIN_HV, J3 VIN_HV, J4 GND, J5 GND, J6 VOUT_LV, J7 VOUT_LV, J8 GND, J9 GND, SW1 SW_REG, U1 AP2112M-8SOIC, U2 TXB0104

Commit message: Finish routing and silkscreen
Parts:
- added REF***: OSHW-Logo_Small_SilkScreen, local_footprints:OSHW-Logo_Small_SilkScreen, B.Cu at (159.9, 89.8)
Routing:
- net 3V3: track 0.00 -> 38.6 mm, vias 0 -> 1
- net 5V: track 0.00 -> 35.6 mm
- net GND: track 0.00 -> 21.7 mm, vias 0 -> 11
- net EN: track 0.00 -> 17.8 mm, vias 0 -> 4
- net Net-(D1-Pad2): track 0.00 -> 7.48 mm
- net L4: track 0.00 -> 5.95 mm
- net H4: track 0.00 -> 5.95 mm
- net L3: track 0.00 -> 4.75 mm
- net H3: track 0.00 -> 4.75 mm
- net L2: track 0.00 -> 3.93 mm
- net H2: track 0.00 -> 3.93 mm
- net L1: track 0.00 -> 3.40 mm
- net H1: track 0.00 -> 3.40 mm
- added copper zone on B.Cu, net GND
- added copper zone on F.Cu, net Net-(D1-Pad2)
Other:
- board text added: "(C) Vlad Belous CC BY-SA 4.0"
- board text added: "3V3"
- board text added: "5V"
- board text added: "AP2112M"
- board text added: "AP2112M + TXB0104"
- board text added: "GND"
- board text added: "H1"
- board text added: "H2"
- board text added: "H3"
- board text added: "H4"
- board text added: "L1"
- board text added: "L2"
- board text added: "L3"
- board text added: "L4"
- board text added: "LDO + logic level shifter"
- board text added: "NOTES:"
- board text added: "TXB0104"
